File: mainboard.sch (EAGLE design)
At the start: 16 parts, among them IC1 7805TV, IC2 7805TV, IC3 7805TV, X1 22-23-2021

Commit message: Add files via upload
Parts:
- removed PERIFERAL: (no value), con-lstb:MA04-1
- removed R3: 120, rcl:R-US_0204/7
- removed U$2: PIN_2X2, DUElib130425:PIN_2X2
- removed V4: ALTIMETER_V4, aero_sensors:ALTIMETER_V4
- added MUX1, MUX2: SN74HC157, QADT:SN74HC157
- added R1: 100k, rcl:R-US_0204/7
- added U$4: ALTIMETER_V5, aero_sensors:ALTIMETER_V5
- G1: device aero_sensors:GPS_ADAFRUIT -> QADT:GPS_ADAFRUIT
- OUT: value PIN_3X8 -> PIN_3X9; device aero_sensors:PIN_3X8 -> QADT:PIN_3X9
- R2: value 120 -> 30k
Connections:
- removed net FLAP_MODE: REC.3.5, U$1.11
- removed net LED_ON: PERIFERAL.4, R3.1
- removed net LED_TEST: R2.2, U$1.50
- removed net LED_TEST_OUT: PERIFERAL.3, R2.1
- removed net LEFT_TAIL: OUT.3.7, U$1.3
- removed net N$1: U$1.GND_1
- removed net N$3: U$2.1.1, XB1.DIN/!CONFIG
- removed net N$4: U$2.1.2, XB1.DOUT
- removed net PID_MODE: REC.3.6, U$1.7
- removed net PITCH_R: REC.3.3, U$1.8
- removed net RIGHT_TAIL: OUT.3.5, U$1.4
- removed net ROLL_R: REC.3.2, U$1.9
- removed net RUDDER: OUT.3.8, U$1.2
- removed net RX1: G1.RX, U$1.RX1
- removed net SPARE: OUT.3.1, U$1.13
- removed net TX1: G1.TX, U$1.TX1
- removed net YAW_R: REC.3.4, U$1.12
- new net BATTERY_VOLTAGE_IN: R1.1, R2.2, U$1.A4
- new net DUE-TO-GPS: G1.RX, U$1.TX1
- new net FLAPS_IN: MUX2.3A, MUX2.4A, REC.3.6, U$1.50
- new net FLAPS_LEFT: MUX2.4Y, OUT.3.8
- new net FLAPS_LEFT_AOUT: MUX2.4B, U$1.7
- new net FLAPS_RIGHT: MUX2.3Y, OUT.3.9
- new net FLAPS_RIGHT_AOUT: MUX2.3B, U$1.8
- new net GPS-TO-DUE: G1.TX, U$1.RX1
- new net LEFT_AILERON_AOUT: MUX1.1B, U$1.5
- new net LEFT_AILERON_IN: MUX1.1A, REC.3.2, U$1.9
- new net LEFT_VTAIL: MUX2.1Y, OUT.3.4
- new net LEFT_VTAIL_AOUT: MUX2.1B, U$1.3
- new net LEFT_VTAIL_IN: MUX2.1A, REC.3.4, U$1.11
- new net RIGHT_AILERON_AOUT: MUX1.2B, U$1.6
- new net RIGHT_AILERON_IN: MUX1.2A, REC.3.3, U$1.10
- new net RIGHT_VTAIL: MUX2.2Y, OUT.3.5
- new net RIGHT_VTAIL_AOUT: MUX2.2B, U$1.4
- new net RIGHT_VTAIL_IN: MUX2.2A, REC.3.5, U$1.12
- new net TAIL_WHEEL: OUT.3.7, U$1.2
- net +5V: now also MUX1.A'/B, MUX2.A'/B; no longer REC.2.1, REC.2.2, REC.2.3, REC.2.4, REC.2.5, REC.2.6, V4.VIN
- net 12V: now also R1.2
- net 3.3V: now also U$4.VIN; no longer R3.2
- net DROP: now also OUT.3.1, U$1.13; no longer OUT.3.2, U$1.10
- net GND: now also MUX1.G', MUX1.GND, MUX2.G', MUX2.GND, OUT.1.9, R2.1, U$1.GND_1, U$4.GND; no longer PERIFERAL.1, V4.GND
- net LEFT_AILERON: now also MUX1.1Y, OUT.3.2; no longer OUT.3.3, U$1.6
- net RESET: no longer PERIFERAL.2
- net RIGHT_AILERON: now also MUX1.2Y, OUT.3.3; no longer OUT.3.4, U$1.5
- net RX: now also XB1.DOUT; no longer U$2.2.2
- net SCL: now also U$4.SCL; no longer V4.SCL
- net SDA: now also U$4.SDA; no longer V4.SDA
- net SERVO_PWR: now also MUX1.VCC, MUX2.VCC, OUT.2.9, REC.2.1, REC.2.2, REC.2.3, REC.2.4, REC.2.5, REC.2.6
- net TX: now also XB1.DIN/!CONFIG; no longer U$2.2.1
Other:
- moved on the sheet: IC1, IC2, IC3, R2, REC, X1-1, X1-2, XB1

Commit message: Add files via upload
Parts:
- OUT: value PIN_3X9 -> PIN_3X10; device QADT:PIN_3X9 -> QADT:PIN_3X10
Connections:
- new net MUX_SELECT_A: MUX1.A'/B, U$1.44
- new net MUX_SELECT_B: MUX2.A'/B, U$1.46
- new net SPARE: OUT.3.10, U$1.9
- net +5V: no longer MUX1.A'/B, MUX2.A'/B
- net GND: now also OUT.1.10; no longer MUX1.G'
- net LEFT_AILERON_IN: now also U$1.40; no longer U$1.9
- net LEFT_VTAIL: now also MUX1.4Y; no longer MUX2.1Y
- net LEFT_VTAIL_AOUT: now also MUX1.4B; no longer MUX2.1B
- net LEFT_VTAIL_IN: now also MUX1.4A, MUX1.G'; no longer MUX2.1A
- net RIGHT_VTAIL: now also MUX1.3Y; no longer MUX2.2Y
- net RIGHT_VTAIL_AOUT: now also MUX1.3B; no longer MUX2.2B
- net RIGHT_VTAIL_IN: now also MUX1.3A; no longer MUX2.2A
- net SERVO_PWR: now also OUT.2.10
