File: mainboard.sch (EAGLE design)
At the start: 16 parts, among them IC1 7805TV, IC2 7805TV, IC3 7805TV, X1 22-23-2021

Commit message: ERC error fixed
Connections:
- net GND: now also MUX1.G'
- net LEFT_VTAIL_IN: no longer MUX1.G'
Changed lines of the file:
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@@
 <part name="GND6" library="supply1" deviceset="GND" device=""/>
 <part name="GND7" library="supply1" deviceset="GND" device=""/>
-<part name="GND9" library="supply1" deviceset="GND" device=""/>
 <part name="R1" library="rcl" deviceset="R-US_" device="0204/7" value="100k"/>
 <part name="R2" library="rcl" deviceset="R-US_" device="0204/7" value="30k"/>
@@
 <part name="GND14" library="supply1" deviceset="GND" device=""/>
 <part name="GND15" library="supply1" deviceset="GND" device=""/>
+<part name="GND9" library="supply1" deviceset="GND" device=""/>
 </parts>
 <sheets>
@@
 <instance part="GND6" gate="1" x="208.28" y="86.36"/>
 <instance part="GND7" gate="1" x="246.38" y="71.12" rot="R90"/>
-<instance part="GND9" gate="1" x="246.38" y="119.38" rot="R90"/>
 <instance part="R1" gate="G$1" x="147.32" y="7.62" rot="R90"/>
 <instance part="R2" gate="G$1" x="147.32" y="-7.62" rot="R90"/>
@@
 <instance part="GND14" gate="1" x="147.32" y="-22.86"/>
 <instance part="GND15" gate="1" x="119.38" y="30.48"/>
+<instance part="GND9" gate="1" x="246.38" y="119.38" rot="R90"/>
 </instances>
 <busses>
@@
 <junction x="119.38" y="38.1"/>
 <pinref part="GND15" gate="1" pin="GND"/>
+</segment>
+<segment>
+<pinref part="MUX1" gate="G$1" pin="G'"/>
+<wire x1="238.76" y1="119.38" x2="243.84" y2="119.38" width="0.1524" layer="91"/>
+<pinref part="GND9" gate="1" pin="GND"/>
 </segment>
 </net>
@@
 </segment>
 <segment>
-<pinref part="MUX1" gate="G$1" pin="G'"/>
-<wire x1="238.76" y1="119.38" x2="243.84" y2="119.38" width="0.1524" layer="91"/>
-<pinref part="GND9" gate="1" pin="GND"/>
-</segment>
-<segment>

Commit message: Board 2016-2017
Parts:
- added DROP, RESET: PUSHBUTTON, QADT:PUSHBUTTON
- added IC4: 7805TV, linear:7805TV
- added LED1, LED2: (no value), led:LED5MM
- added R3, R4: 200, rcl:R-US_0204/7
- added R5, R6: 2k, rcl:R-US_0204/7
- U$4: device aero_sensors:ALTIMETER_V5 -> QADT:ALTIMETER_V5
Connections:
- removed net A0: U$1.A0
- new net DROP_BUTTON: DROP.1, R6.2, U$1.13
- new net FIX: R3.2, U$1.A10
- new net N$1: LED1.A, R3.1
- new net N$3: LED2.A, R4.1
- new net RESET_BUTTON: R5.2, RESET.1, U$1.48
- new net STATUS: R4.2, U$1.A11
- net 12V: now also IC4.VI
- net 3.3V: now also DROP.2, RESET.2
- net DROP: now also U$1.10; no longer U$1.13
- net GND: now also IC4.GND, LED1.C, LED2.C, R5.1, R6.1
- net RIGHT_AILERON_IN: now also U$1.42; no longer U$1.10
- net SERVO_PWR: now also IC4.VO
