File: mainboard.brd (EAGLE design)
At the start: 104.6 x 57.8 mm, 16 parts, among them IC1 7805TV, IC2 7805TV, IC3 7805TV, X1 22-23-2021

Commit message: Board 2016-2017
Parts:
- added DROP, RESET: PUSHBUTTON, QADT:PUSHBUTTON
- added IC4: 7805TV, linear:TO220V
- added LED1, LED2: (no value), led:LED5MM
- added R3, R4: 200, rcl:0204/7
- added R5, R6: 2k, rcl:0204/7
- U$4: device aero_sensors:ALTIMETER_V5 -> QADT:ALTIMETER_V5
- moved IC3 4.51 mm to (42.0, 16.0)
- moved IC2 2.41 mm to (36.3, 16.0)
- moved G1 0.76 mm to (46.0, 39.1)
- moved MPU 0.76 mm to (65.8, 23.7)
- moved MUX1 0.76 mm to (34.2, 44.3)
- moved MUX2 0.76 mm to (43.1, 30.9)
- moved OUT 0.76 mm to (13.1, 18.4)
- moved R1 0.76 mm to (65.8, 20.1)
- moved REC 0.76 mm to (14.0, 49.8)
- moved U$1 0.76 mm to (78.2, 23.9)
- moved U$4 0.76 mm to (87.6, 9.78)
- moved X1 0.76 mm to (24.3, 7.11)
- moved XB1 0.76 mm to (82.2, 39.2)
- moved U$3 0.76 mm to (8.13, 5.84)
- moved IC1 0.76 mm to (30.2, 16.0)
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Connections:
- removed net A0: U$1.A0
- new net DROP_BUTTON: DROP.1, R6.2, U$1.13
- new net FIX: R3.2, U$1.A10
- new net N$1: LED1.A, R3.1
- new net N$3: LED2.A, R4.1
- new net RESET_BUTTON: R5.2, RESET.1, U$1.48
- new net STATUS: R4.2, U$1.A11
- net 12V: now also IC4.1
- net 3.3V: now also DROP.2, RESET.2
- net DROP: now also U$1.10; no longer U$1.13
- net GND: now also IC4.2, LED1.K, LED2.K, R5.1, R6.1
- net RIGHT_AILERON_IN: now also U$1.42; no longer U$1.10
- net SERVO_PWR: now also IC4.3
Routing:
- net FIX: track 0.00 -> 175.7 mm, vias 0 -> 1
- net STATUS: track 0.00 -> 159.1 mm, vias 0 -> 2
- net RIGHT_AILERON_IN: track 63.4 -> 199.6 mm, vias 3 -> 7
- net 3.3V: track 131.0 -> 262.6 mm, vias 0 -> 6
- net RESET_BUTTON: track 0.00 -> 119.3 mm, vias 0 -> 2
- net GND: track 316.3 -> 414.2 mm, vias 3 -> 6
- net SERVO_PWR: track 174.1 -> 113.3 mm, vias 3 -> 0
- net N$3: track 0.00 -> 39.6 mm
- net DROP_BUTTON: track 0.00 -> 35.2 mm
- net N$1: track 0.00 -> 14.7 mm
- net DROP: track 65.6 -> 80.1 mm
- net LEFT_AILERON_IN: track 187.6 -> 192.6 mm
- net FLAPS_IN: track 197.5 -> 202.3 mm
- net RIGHT_VTAIL: track 44.6 -> 49.3 mm
- net LEFT_VTAIL: track 147.3 -> 149.4 mm
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Other:
- board size 104.6 x 57.8 mm -> 106 x 68.7 mm
- board text added: "!FIX"
- board text added: "13"
- board text added: "2"
- board text added: "3.3V"
- board text added: "40"
- board text added: "42"
- board text added: "52"
- board text added: "5V"
- board text added: "A11"
- board text added: "DROP"
- board text added: "PWM"
- board text added: "RESET"
- board text added: "RX0"
- board text added: "RX1"
- board text added: "RX2"
- board text added: "RX3"
- board text added: "SCL1"
- board text added: "SDA1"
- board text added: "STATUS"
- board text added: "TX0"
- board text added: "TX1"
- board text added: "TX2"
- board text added: "TX3"
